File: ControlRTC.kicad_sch (KiCad schematic)
At the start: 30 parts, among them J701 Molex 470531000, U21 PCF85063AT, U701 74LVC1G07, U702 EMC2301-1-ACZL-TR, Y2 32768Hz{slash}12.5pF

Commit message: Weeded out all ERC errors
Parts:
- removed C706: 100n, Capacitor_SMD:C_0402_1005Metric, symbol Device:C_Small
- removed C707: 100n, Capacitor_SMD:C_0402_1005Metric, symbol Device:C
- removed D703: LED Red, LED_SMD:LED_0603_1608Metric, symbol Device:LED_Small
- removed D704: LED Green, LED_SMD:LED_0603_1608Metric, symbol Device:LED_Small
- removed JP701: Bridged, Jumper:SolderJumper-2_P1.3mm_Bridged2Bar_Pad1.0x1.5mm, symbol Jumper:SolderJumper_2_Bridged
- removed R38: 100R, Resistor_SMD:R_0402_1005Metric, symbol Device:R_Small
- removed R702: 1k, Resistor_SMD:R_0402_1005Metric, symbol Device:R_Small
- removed R703: 22k/1%, Resistor_SMD:R_0402_1005Metric, symbol Device:R_Small
- removed R704: 36K 1%, Resistor_SMD:R_0402_1005Metric, symbol Device:R
- removed TP11, TP12, TP13: TestPoint, TestPoint:TestPoint_Pad_D1.0mm, symbol Connector:TestPoint
- removed U21: PCF85063AT, Package_SO:SOIC-8_3.9x4.9mm_P1.27mm, symbol Timer_RTC:PCF8563T
- removed U701: 74LVC1G07, Package_TO_SOT_SMD:SOT-23-5, symbol 74xGxx:74LVC1G07
- removed U702: EMC2301-1-ACZL-TR, Package_SO:MSOP-8_3x3mm_P0.65mm, symbol CM4IO:EMC2301
- removed Y2: 32768Hz/12.5pF, Crystal:Crystal_SMD_3215-2Pin_3.2x1.5mm, symbol Device:Crystal_Small
- added C708: 22pF C0G, Capacitor_SMD:C_0603_1608Metric, symbol Device:C_Small
- added J702: HC-1.0-4PLT, Hatlabs:JST_SH_HCTL_HC-1.0-4PLT_1x04-1MP_P1.00mm_Vertical, symbol Connector_Generic:Conn_01x04
- added JP701: Jumper_2_Bridged, Connector_PinHeader_2.54mm:PinHeader_1x02_P2.54mm_Vertical, symbol Jumper:Jumper_2_Bridged
- added U702: PCF85063ATL, Package_DFN_QFN:DFN-10-1EP_2.6x2.6mm_P0.5mm_EP1.3x2.2mm, symbol Timer_RTC:PCF85063ATL
- added Y701: X1A000061000200, Crystal:Crystal_SMD_2012-2Pin_2.0x1.2mm, symbol Device:Crystal
- BT701: renamed from BT1; value Battery_Cell -> BS-02-A1AJ010; footprint Battery:BatteryHolder_Keystone_1060_1x2032 -> Battery:BatteryHolder_MYOUNG_BS-07-A1BJ001_CR2032; LCSC (none) -> C5239862; Manufacturer Keystone -> (none); PartNumber 1060 -> (none)
- C702: renamed from C711; value 100n -> 100nF; LCSC (none) -> C1525
- C703: renamed from C712; LCSC (none) -> C52923
- C704: renamed from C710; value 100n -> 100nF; LCSC (none) -> C1525
- C705: renamed from C709; LCSC (none) -> C52923
- C706: renamed from C708; LCSC (none) -> C23733
- C707: renamed from C68; value 100n -> 100nF; LCSC (none) -> C1525
- D703: renamed from D24; value BAT54C-7-F -> BAT54C,215; LCSC (none) -> C37704
- J701: Field4 Farnell -> (none); Field5 2313705 -> (none); Field6 470531000 -> (none); Field7 Molex -> (none); LCSC (none) -> C2982033; Part Description Connector Header Through Hole 4 position 0.100" (2.54mm) -> (none)
- LED701, LED702, LED703, LED704, LED705: value Worldsemi_WS2812E-4020 -> SK6805MICRO-J; footprint Hatlabs:LED_WS2812E-4020_PLCC4_4.0x2.0mm_P0.85mm -> LED_SMD:LED_SK6805_PLCC4_2.4x2.7mm_P1.3mm; LCSC (none) -> C2909056
Connections:
- net +3V3: now also D703.1
- net +5V: now also C702.1, C703.1, LED701.1 (VCC), LED702.1 (VCC), LED703.1 (VCC), LED704.1 (VCC), LED705.1 (VCC), J702.1 (Pin_1)
- net GND: now also C708.1, J702.3 (Pin_3), U702.3 (CLKOE), U702.5 (VSS)
- net I2C0.SCL: now also U702.7 (SCL)
- net I2C0.SDA: now also U702.6 (SDA)
- net RTC_INT: now also U702.4 (~{INT})
- net at D703.3: now also JP701.1 (A)
- net at C707.1: now also JP701.2 (B), U702.10 (VDD)
- net VBAT: now reaches BT701.1 (+), C706.1
- net VBAT: now also D703.2
- net FAN_TACHO: now reaches J701.3 (Pin_3)
- net FAN_TACHO: now also J702.4 (Pin_4)
- net FAN_PWM: now reaches J701.4 (Pin_4)
- net FAN_PWM: now also J702.2 (Pin_2)
- removed net +3.3VP: C702.1, C703.1, D703.1, LED701.1 (VCC), LED702.1 (VCC), LED703.1 (VCC), LED704.1 (VCC), LED705.1 (VCC)
- new net: U702.2 (OSCO), Y701.1
- new net: C708.2, U702.1 (OSCI), Y701.2
- no-connect marks 4 -> 2
Other:
- note added: "CM5 FAN connector"
- note added: "FAN connectors"
- note added: "Provide both a Pi 5 style and an old-school Molex fan connector"
- note added: "Remove the jumper cap to disable the RTC"
- note added: "Yellow FAN connector"
- note removed: "Also SMBUS alert IIC address : 0001_100x"
- note removed: "Cut the solder jumper to disable the RTC"
- note removed: "FAN connector"
- note removed: "FAN controller"
- note removed: "IIC address : 0101_111x"
- note removed: "Power and ACT LEDs"
- company: Nabu Casa -> Hat Labs Oy
- title: Control/RTC -> HALPI2
- moved on the sheet: C704, C705, J701

Commit message: Re-annotate schematics
Parts:
- renumbered C702 to C701, C703 to C702, C704 to C703, C705 to C704, C706 to C705, C707 to C706, C708 to C707, D703 to D701, U702 to U701

Commit message: Sprinkle test points on the schematics
Parts:
- added TP701, TP702: TestPoint, TestPoint:TestPoint_Pad_D1.0mm, symbol Connector:TestPoint
Connections:
- net FAN_TACHO: now also TP701.1
- net RTC_INT: now also TP702.1

Commit message: Implement a USB3 hub
Connections:
- net +3V3 renamed +3.3V
Changed lines of the file:
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@@
 	)
 	(symbol
-		(lib_id "power:+3V3")
+		(lib_id "power:+3.3V")
 		(at 189.23 105.41 0)
 		(unit 1)
@@
 			)
 		)
-		(property "Value" "+3V3"
-			(at 189.23 100.584 0)
+		(property "Value" "+3.3V"
+			(at 189.23 101.854 0)
 			(effects
 				(font
@@
 			)
 		)
-		(property "Description" "Power symbol creates a global label with name \"+3V3\""
+		(property "Description" "Power symbol creates a global label with name \"+3.3V\""
 			(at 189.23 105.41 0)
 			(effects
@@
 			)
 		)
+		(property "Sim.Enable" ""
+			(at 81.28 168.91 0)
+			(effects
+				(font
+					(size 1.27 1.27)
+				)
+				(hide yes)
+			)
+		)
 		(pin "1"
 		)
@@
 			(at 262.89 134.62 0)
 			(effects
+				(font
+					(size 1.27 1.27)
+				)
+				(hide yes)
+			)
+		)
+		(property "Sim.Enable" ""
+			(at 262.89 134.62 0)
+			(effects
