File: SDCard.kicad_sch (KiCad schematic)
At the start: 5 parts, among them J7 Micro_SD_Card_Det, U22 RT9742GGJ5

Commit message: Weeded out all ERC errors
Parts:
- removed C72: 10u, Capacitor_SMD:C_0805_2012Metric, symbol Device:C_Small
- removed R39, R40: 10k, Resistor_SMD:R_0402_1005Metric, symbol Device:R_Small
- removed U22: RT9742GGJ5, Package_TO_SOT_SMD:SOT-23-5, symbol Yellow:RT9742GGJ5
- added C804, C806: 10uF, Capacitor_SMD:C_0805_2012Metric, symbol Device:C_Small
- added C805: 100nF, Capacitor_SMD:C_0402_1005Metric, symbol Device:C_Small
- added R806: 49.9k, Resistor_SMD:R_0603_1608Metric, symbol Device:R_Small
- added U801: AP22653W6-7, Package_TO_SOT_SMD:SOT-23-6, symbol Hatlabs:AP22653
- J801: renamed from J7; footprint Connector_Card:microSD_HC_Molex_104031-0811 -> Hatlabs:MicroSD_SHOU-HAN_TF-PUSH; symbol Connector:Micro_SD_Card_Det -> Connector:Micro_SD_Card_Det1; LCSC (none) -> C393941; Manufacturer Molex -> SHOU HAN; PartNumber 104031-0811 -> TF PUSH
Connections:
- net +3V3 is gone; now on net GND: J801.10 (SHIELD)
- net GND: now also C804.2, C805.2, C806.2, R806.1, U801.2 (GND); no longer J801.11 (SHIELD)
- net SD.PWR: now also U801.3 (EN)
- net SD_+3V3: now also C806.1, U801.6 (OUT)
- new net: R806.2, U801.5 (ILIM)
- new net CMx_3V3: C804.1, C805.1, U801.1 (IN)
- no-connect marks 1 -> 2
Other:
- company: Nabu Casa -> Hat Labs Oy
- title: SD card -> HALPI2

Commit message: Implement ideal diodes for input and LDO power ORing
Other:
- note added: "Current limiting"
- moved on the sheet: C804, C805, C806, R806, U801

Commit message: Re-annotate schematics
Parts:
- renumbered C804 to C801, C805 to C802, C806 to C803, R806 to R801
Changed lines of the file:
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@@
 		(dnp no)
 		(fields_autoplaced yes)
-		(property "Reference" "R806"
+		(property "Reference" "R801"
 			(at 77.47 138.4299 0)
 			(effects
@@
 			)
 		)
-		(property "Sim.Enable" ""
-			(at 80.01 140.97 0)
-			(effects
-				(font
-					(size 1.27 1.27)
-				)
-				(hide yes)
-			)
-		)
 		(pin "1"
 		)
@@
 			(project "HALPI2"
 				(path "/abc482bd-3f17-4d35-80db-1da3dcdb5c27/67ada73c-6692-4fd8-8c20-5be89f2b8650"
-					(reference "R806")
+					(reference "R801")
 					(unit 1)
 				)
@@
 			)
 		)
-		(property "Sim.Enable" ""
-			(at 102.87 71.12 0)
-			(effects
-				(font
-					(size 1.27 1.27)
-				)
-				(hide yes)
-			)
-		)
 		(pin "1"
 		)
@@
 		(on_board yes)
 		(dnp no)
-		(property "Reference" "#PWR0811"
+		(property "Reference" "#PWR0801"
 			(at 76.2 125.73 0)
 			(effects
@@
 			(project "HALPI2"
 				(path "/abc482bd-3f17-4d35-80db-1da3dcdb5c27/67ada73c-6692-4fd8-8c20-5be89f2b8650"
-					(reference "#PWR0811")
+					(reference "#PWR0801")
 					(unit 1)
 				)
@@
 		(dnp no)
 		(fields_autoplaced yes)
-		(property "Reference" "C805"
+		(property "Reference" "C802"
 			(at 83.82 113.0362 0)
 			(effects
@@
 			)
 		)
-		(property "Sim.Enable" ""
-			(at 81.28 115.57 0)
-			(effects
-				(font
-					(size 1.27 1.27)
-				)
-				(hide yes)
-			)
-		)
 		(pin "1"
 		)
@@
 			(project "HALPI2"
 				(path "/abc482bd-3f17-4d35-80db-1da3dcdb5c27/67ada73c-6692-4fd8-8c20-5be89f2b8650"
-					(reference "C805")
+					(reference "C802")
 					(unit 1)
 				)
@@
 		(on_board yes)
 		(dnp no)
-		(property "Reference" "C806"
+		(property "Reference" "C803"
 			(at 120.65 133.35 0)
 			(effects
@@
 			)
 		)
-		(property "Sim.Enable" ""
-			(at 118.11 134.62 0)
-			(effects
-				(font
-					(size 1.27 1.27)
-				)
-				(hide yes)
-			)
-		)
 		(pin "1"
 		)
@@
 			(project "HALPI2"
 				(path "/abc482bd-3f17-4d35-80db-1da3dcdb5c27/67ada73c-6692-4fd8-8c20-5be89f2b8650"
-					(reference "C806")
+					(reference "C803")
 					(unit 1)
 				)
@@
 		(on_board yes)
 		(dnp no)
-		(property "Reference" "#PWR0815"
+		(property "Reference" "#PWR0806"
 			(at 97.79 148.59 0)
 			(effects
@@
 			(project "HALPI2"
 				(path "/abc482bd-3f17-4d35-80db-1da3dcdb5c27/67ada73c-6692-4fd8-8c20-5be89f2b8650"
-					(reference "#PWR0815")
+					(reference "#PWR0806")
 					(unit 1)
 				)
@@
 		(on_board yes)
 		(dnp no)
-		(property "Reference" "#PWR0816"
+		(property "Reference" "#PWR0803"
 			(at 80.01 152.4 0)
 			(effects
@@
 			(project "HALPI2"
 				(path "/abc482bd-3f17-4d35-80db-1da3dcdb5c27/67ada73c-6692-4fd8-8c20-5be89f2b8650"
-					(reference "#PWR0816")
+					(reference "#PWR0803")
 					(unit 1)
 				)
@@
 		(on_board yes)
 		(dnp no)
-		(property "Reference" "C804"
+		(property "Reference" "C801"
 			(at 73.66 113.0362 0)
 			(effects
@@
 			)
 		)
-		(property "Sim.Enable" ""
-			(at 76.2 115.57 0)
-			(effects
-				(font
-					(size 1.27 1.27)
-				)
-				(hide yes)
-			)
-		)
 		(pin "1"
 		)
@@
 			(project "HALPI2"
 				(path "/abc482bd-3f17-4d35-80db-1da3dcdb5c27/67ada73c-6692-4fd8-8c20-5be89f2b8650"
-					(reference "C804")
+					(reference "C801")
 					(unit 1)
 				)
@@
 		(on_board yes)
 		(dnp no)
-		(property "Reference" "#PWR0814"
+		(property "Reference" "#PWR0807"
 			(at 118.11 146.05 0)
 			(effects
@@
 			(project "HALPI2"
 				(path "/abc482bd-3f17-4d35-80db-1da3dcdb5c27/67ada73c-6692-4fd8-8c20-5be89f2b8650"
-					(reference "#PWR0814")
+					(reference "#PWR0807")
 					(unit 1)
 				)
@@
 		(on_board yes)
 		(dnp no)
-		(property "Reference" "#PWR0812"
+		(property "Reference" "#PWR0804"
 			(at 81.28 125.73 0)
 			(effects
@@
 			(project "HALPI2"
 				(path "/abc482bd-3f17-4d35-80db-1da3dcdb5c27/67ada73c-6692-4fd8-8c20-5be89f2b8650"
-					(reference "#PWR0812")
+					(reference "#PWR0804")
 					(unit 1)
 				)
@@
 		(on_board yes)
 		(dnp no)
-		(property "Reference" "#PWR0813"
+		(property "Reference" "#PWR0805"
 			(at 86.36 114.3 0)
 			(effects
@@
 			(project "HALPI2"
 				(path "/abc482bd-3f17-4d35-80db-1da3dcdb5c27/67ada73c-6692-4fd8-8c20-5be89f2b8650"
-					(reference "#PWR0813")
-					(unit 1)
-				)
+					(reference "#PWR0805")
+					(unit 1)
+				)

Commit message: Sprinkle test points on the schematics
Parts:
- added TP801: TestPoint, TestPoint:TestPoint_Pad_D1.0mm, symbol Connector:TestPoint
Connections:
- net SD_+3V3: now also TP801.1
Changed lines of the file:
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@@
+	)
+	(junction
+		(at 111.76 128.27)
+		(diameter 0)
+		(color 0 0 0 0)
 	)
 	(junction
@@
 	(wire
 		(pts
-			(xy 109.22 128.27) (xy 118.11 128.27)
+			(xy 109.22 128.27) (xy 111.76 128.27)
 		)
 		(stroke
@@
 			(width 0)
 			(type default)
+		)
+	)
+	(wire
+		(pts
+			(xy 111.76 128.27) (xy 118.11 128.27)
+		)
+		(stroke
+			(width 0)
+			(type solid)
 		)
 	)
@@
 			)
 		)
+		(property "Sim.Enable" ""
+			(at 80.01 140.97 0)
+			(effects
+				(font
+					(size 1.27 1.27)
+				)
+				(hide yes)
+			)
+		)
 		(pin "1"
 		)
@@
 		)
 		(property "LCSC" "C393941"
+			(at 102.87 71.12 0)
+			(effects
+				(font
+					(size 1.27 1.27)
+				)
+				(hide yes)
+			)
+		)
+		(property "Sim.Enable" ""
 			(at 102.87 71.12 0)
 			(effects
@@
 			)
 		)
+		(property "Sim.Enable" ""
+			(at 97.79 132.08 0)
+			(effects
+				(font
+					(size 1.27 1.27)
+				)
+				(hide yes)
+			)
+		)
 		(pin "2"
 		)
@@
 			)
 		)
+		(property "Sim.Enable" ""
+			(at 81.28 115.57 0)
+			(effects
+				(font
+					(size 1.27 1.27)
+				)
+				(hide yes)
+			)
+		)
 		(pin "1"
 		)
@@
 				(path "/abc482bd-3f17-4d35-80db-1da3dcdb5c27/67ada73c-6692-4fd8-8c20-5be89f2b8650"
 					(reference "C802")
+					(unit 1)
+				)
+			)
+		)
+	)
+	(symbol
+		(lib_id "Connector:TestPoint")
+		(at 111.76 128.27 0)
+		(mirror y)
+		(unit 1)
+		(exclude_from_sim no)
+		(in_bom yes)
+		(on_board yes)
+		(dnp no)
+		(property "Reference" "TP801"
+			(at 114.3 126.2381 0)
+			(effects
+				(font
+					(size 1.27 1.27)
+				)
+				(justify right)
+			)
+		)
+		(property "Value" "TestPoint"
+			(at 114.3 123.6981 0)
+			(effects
+				(font
+					(size 1.27 1.27)
+				)
+				(justify right)
+			)
+		)
+		(property "Footprint" "TestPoint:TestPoint_Pad_D1.0mm"
+			(at 106.68 128.27 0)
+			(effects
+				(font
+					(size 1.27 1.27)
+				)
+				(hide yes)
+			)
+		)
+		(property "Datasheet" "~"
+			(at 106.68 128.27 0)
+			(effects
+				(font
+					(size 1.27 1.27)
+				)
+				(hide yes)
+			)
+		)
+		(property "Description" "test point"
+			(at 111.76 128.27 0)
+			(effects
+				(font
+					(size 1.27 1.27)
+				)
+				(hide yes)
+			)
+		)
+		(pin "1"
+		)
+		(instances
+			(project "HALPI2"
+				(path "/abc482bd-3f17-4d35-80db-1da3dcdb5c27/67ada73c-6692-4fd8-8c20-5be89f2b8650"
+					(reference "TP801")
 					(unit 1)
 				)
@@
 		)
 		(property "LCSC" "C15850"
+			(at 118.11 134.62 0)
+			(effects
+				(font
+					(size 1.27 1.27)
+				)
+				(hide yes)
+			)
+		)
+		(property "Sim.Enable" ""
 			(at 118.11 134.62 0)
 			(effects
@@
 			)
 		)
+		(property "Sim.Enable" ""
+			(at 76.2 115.57 0)
+			(effects
+				(font
+					(size 1.27 1.27)
+				)
+				(hide yes)
+			)
+		)

Commit message: Fix ethernet port & other changes
Changed lines of the file:
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@@
 		(pin "5"
 		)
-		(pin ""
+		(pin "4"
 		)
 		(pin "3"

Commit message: Implement a USB3 hub
Connections:
- net CMx_3V3 renamed +3.3VCMx
Changed lines of the file:
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@@
+			)
+		)
+		(property "Sim.Enable" ""
+			(at 111.76 128.27 0)
+			(effects
+				(font
+					(size 1.27 1.27)
+				)
+				(hide yes)
 			)
 		)
@@
 	)
 	(symbol
-		(lib_id "power:+3V3")
+		(lib_id "Hatlabs:+3.3VCMx")
 		(at 86.36 110.49 0)
 		(unit 1)
@@
 			)
 		)
-		(property "Value" "CMx_3V3"
+		(property "Value" "+3.3VCMx"
 			(at 86.36 106.934 0)
 			(effects
@@
 			)
 		)
-		(property "Description" "Power symbol creates a global label with name \"+3V3\""
+		(property "Description" "Power symbol driven by the CMx module +3.3V output"
 			(at 86.36 110.49 0)
 			(effects

Commit message: Partial trace layout, kick-ass custom rules
Parts:
- renumbered C801 to C1001, C802 to C1002, C803 to C1003, J801 to J1001, R801 to R1001, TP801 to TP1001, U801 to U1001
Connections:
- net ILIM: now reaches R1001.2, U1001.5 (ILIM)
- net +3.3VCMx renamed +3.3V
- net SD_+3V3 renamed +3.3VSD

Commit message: A big part of layout and routing done
Parts:
- C1001, C1002, C1003, R1001, U1001: Config +SDCard -> (none)
- J1001: Config +SDCard -> (none); Manufacturer SHOU HAN -> (none); PartNumber TF PUSH -> (none)
