File: idc.kicad_sch (KiCad schematic)
At the start: 3 parts, among them Q2101 MMDT5401

Commit message: Re-annotate schematics
Parts:
- renumbered Q2101 to Q2102
Connections:
- net CATHODE: now also Q2102.6 (C1); no longer Q2102.3 (C2)
- net GATE: now also Q2102.1 (E1); no longer Q2102.4 (E2)
- net at Q2101.1 (E1), Q2101.2 (B1), R2101.2: now also Q2102.2 (B1); no longer Q2102.5 (B2)
Changed lines of the file:
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@@
 		(pin "1"
+		)
+		(instances
+			(project "HALPI2"
+				(path "/abc482bd-3f17-4d35-80db-1da3dcdb5c27/850df4bf-e40a-4082-adc2-76804638b949/941fe792-02c8-46de-a01c-95bb6b865738"
+					(reference "R2101")
+					(unit 1)
+				)
+			)
 		)
 	)
@@
 		(lib_id "Transistor_BJT:MMDT5401")
 		(at 152.4 92.71 0)
-		(unit 2)
+		(unit 1)
 		(exclude_from_sim no)
 		(in_bom yes)
@@
 		(dnp no)
 		(fields_autoplaced yes)
-		(property "Reference" "Q2101"
+		(property "Reference" "Q2102"
 			(at 157.48 91.4399 0)
 			(effects
@@
 		(pin "5"
 		)
+		(instances
+			(project "HALPI2"
+				(path "/abc482bd-3f17-4d35-80db-1da3dcdb5c27/850df4bf-e40a-4082-adc2-76804638b949/941fe792-02c8-46de-a01c-95bb6b865738"
+					(reference "Q2102")
+					(unit 1)
+				)
+			)
+		)
 	)

Commit message: Sprinkle test points on the schematics
Parts:
- added TP2101: TestPoint, TestPoint:TestPoint_Pad_D1.0mm, symbol Connector:TestPoint
- R2101: footprint (none) -> Resistor_SMD:R_0402_1005Metric; LCSC (none) -> C25744
- R2102: footprint (none) -> Resistor_SMD:R_0402_1005Metric; LCSC (none) -> C25792
Connections:
- net GATE: now also TP2101.1
Changed lines of the file:
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@@
+	)
+	(junction
+		(at 154.94 100.33)
+		(diameter 0)
+		(color 0 0 0 0)
 	)
 	(junction
@@
 	(wire
 		(pts
-			(xy 154.94 97.79) (xy 154.94 102.87)
+			(xy 154.94 100.33) (xy 154.94 102.87)
+		)
+		(stroke
+			(width 0)
+			(type default)
+		)
+	)
+	(wire
+		(pts
+			(xy 154.94 97.79) (xy 154.94 100.33)
 		)
 		(stroke
@@
 			)
 			(justify left)
+		)
+	)
+	(symbol
+		(lib_id "Connector:TestPoint")
+		(at 154.94 100.33 270)
+		(mirror x)
+		(unit 1)
+		(exclude_from_sim no)
+		(in_bom yes)
+		(on_board yes)
+		(dnp no)
+		(fields_autoplaced yes)
+		(property "Reference" "TP2101"
+			(at 160.02 99.0599 90)
+			(effects
+				(font
+					(size 1.27 1.27)
+				)
+				(justify left)
+			)
+		)
+		(property "Value" "TestPoint"
+			(at 160.02 101.5999 90)
+			(effects
+				(font
+					(size 1.27 1.27)
+				)
+				(justify left)
+			)
+		)
+		(property "Footprint" "TestPoint:TestPoint_Pad_D1.0mm"
+			(at 154.94 95.25 0)
+			(effects
+				(font
+					(size 1.27 1.27)
+				)
+				(hide yes)
+			)
+		)
+		(property "Datasheet" "~"
+			(at 154.94 95.25 0)
+			(effects
+				(font
+					(size 1.27 1.27)
+				)
+				(hide yes)
+			)
+		)
+		(property "Description" "test point"
+			(at 154.94 100.33 0)
+			(effects
+				(font
+					(size 1.27 1.27)
+				)
+				(hide yes)
+			)
+		)
+		(pin "1"
+		)
+		(instances
+			(project "HALPI2"
+				(path "/abc482bd-3f17-4d35-80db-1da3dcdb5c27/850df4bf-e40a-4082-adc2-76804638b949/941fe792-02c8-46de-a01c-95bb6b865738"
+					(reference "TP2101")
+					(unit 1)
+				)
+			)
 		)
 	)
@@
 			)
 		)
-		(property "Footprint" ""
+		(property "Footprint" "Resistor_SMD:R_0402_1005Metric"
 			(at 154.94 109.22 0)
 			(effects
@@
 		)
 		(property "Description" "Resistor, small symbol"
+			(at 154.94 109.22 0)
+			(effects
+				(font
+					(size 1.27 1.27)
+				)
+				(hide yes)
+			)
+		)
+		(property "Sim.Enable" ""
+			(at 154.94 109.22 0)
+			(effects
+				(font
+					(size 1.27 1.27)
+				)
+				(hide yes)
+			)
+		)
+		(property "LCSC" "C25792"
 			(at 154.94 109.22 0)
 			(effects
@@
 			)
 		)
-		(property "Footprint" ""
+		(property "Footprint" "Resistor_SMD:R_0402_1005Metric"
 			(at 134.62 109.22 0)
 			(effects
@@
 		)
 		(property "Description" "Resistor, small symbol"
+			(at 134.62 109.22 0)
+			(effects
+				(font
+					(size 1.27 1.27)
+				)
+				(hide yes)
+			)
+		)
+		(property "Sim.Enable" ""
+			(at 134.62 109.22 0)
+			(effects
+				(font
+					(size 1.27 1.27)
+				)
+				(hide yes)
+			)
+		)
+		(property "LCSC" "C25744"
 			(at 134.62 109.22 0)
 			(effects
@@
 			)
 		)
+		(property "Sim.Enable" ""
+			(at 137.16 92.71 0)
+			(effects
+				(font
+					(size 1.27 1.27)
+				)
+				(hide yes)
+			)
+		)
 		(pin "4"
 		)
@@
 			(at 152.4 92.71 0)
 			(effects
+				(font
+					(size 1.27 1.27)
+				)
+				(hide yes)
+			)
+		)
+		(property "Sim.Enable" ""
+			(at 152.4 92.71 0)
+			(effects

Commit message: Implement a USB3 hub
Parts:
- renumbered Q2101 to Q?
Changed lines of the file:
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@@
+			)
+		)
+		(property "Sim.Enable" ""
+			(at 154.94 100.33 0)
+			(effects
+				(font
+					(size 1.27 1.27)
+				)
+				(hide yes)
 			)
 		)
@@
 			)
 		)
-		(property "Sim.Enable" ""
-			(at 154.94 109.22 0)
-			(effects
-				(font
-					(size 1.27 1.27)
-				)
-				(hide yes)
-			)
-		)
 		(property "LCSC" "C25792"
+			(at 154.94 109.22 0)
+			(effects
+				(font
+					(size 1.27 1.27)
+				)
+				(hide yes)
+			)
+		)
+		(property "Sim.Enable" ""
 			(at 154.94 109.22 0)
 			(effects
@@
 			)
 		)
-		(property "Sim.Enable" ""
-			(at 134.62 109.22 0)
-			(effects
-				(font
-					(size 1.27 1.27)
-				)
-				(hide yes)
-			)
-		)
 		(property "LCSC" "C25744"
+			(at 134.62 109.22 0)
+			(effects
+				(font
+					(size 1.27 1.27)
+				)
+				(hide yes)
+			)
+		)
+		(property "Sim.Enable" ""
 			(at 134.62 109.22 0)
 			(effects
@@
 		(on_board yes)
 		(dnp no)
-		(property "Reference" "Q2101"
+		(property "Reference" "Q?"
 			(at 132.08 91.4399 0)
 			(effects
@@
 		)
 		(instances
-			(project ""
-				(path "/abc482bd-3f17-4d35-80db-1da3dcdb5c27/850df4bf-e40a-4082-adc2-76804638b949/941fe792-02c8-46de-a01c-95bb6b865738"
-					(reference "Q2101")
-					(unit 1)
-				)
+			(project "HALPI2"
+				(path "/abc482bd-3f17-4d35-80db-1da3dcdb5c27/850df4bf-e40a-4082-adc2-76804638b949/941fe792-02c8-46de-a01c-95bb6b865738"
+					(reference "Q?")
+					(unit 1)
+				)

Commit message: Finish component selection for USB3 hub
Parts:
- Q2102, Q?: LCSC (none) -> C2919802
Changed lines of the file:
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@@
+			)
+		)
+		(property "LCSC" "C2919802"
+			(at 137.16 92.71 0)
+			(effects
+				(font
+					(size 1.27 1.27)
+				)
+				(hide yes)
 			)
 		)
@@
 			(at 152.4 92.71 0)
 			(effects
+				(font
+					(size 1.27 1.27)
+				)
+				(hide yes)
+			)
+		)
+		(property "LCSC" "C2919802"
+			(at 152.4 92.71 0)
+			(effects

Commit message: Partial trace layout, kick-ass custom rules
Parts:
- removed Q2102, Q?: MMDT5401, Package_TO_SOT_SMD:SOT-363_SC-70-6, symbol Transistor_BJT:MMDT5401
- removed TP2101: TestPoint, TestPoint:TestPoint_Pad_D1.0mm, symbol Connector:TestPoint
- added Q2401: MMDT5401, Package_TO_SOT_SMD:SOT-363_SC-70-6, symbol Transistor_BJT:MMDT5401
- renumbered R2101 to R2401, R2102 to R2402
Connections:
- net ANODE: now also Q2401.1 (E1)
- net CATHODE: now also Q2401.4 (E2)
- net GATE: now also Q2401.3 (C2)
- net B: now reaches R2401.2
- net B: now also Q2401.2 (B1), Q2401.5 (B2), Q2401.6 (C1)

Commit message: A big part of layout and routing done
Parts:
- Q2401: LCSC (none) -> C2919802
Changed lines of the file:
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@@
 (kicad_sch
-	(version 20231120)
+	(version 20250114)
 	(generator "eeschema")
-	(generator_version "8.0")
+	(generator_version "9.0")
 	(paper "A4")
 	(title_block
@@
 		(comment 3 "HALPI2 is licensed under CC BY 4.0.")
 	)
+	(text "Ideal diode controller\n\nUse a P-channel MOSFET as an ideal diode\nwith a very low voltage drop while maintaining\nreverse voltage protection and reverse current\nblocking."
+		(exclude_from_sim no)
+		(at 64.516 100.838 0)
+		(effects
+			(font
+				(size 1.27 1.27)
+			)
+			(justify left)
+		)
+	)
+	(text "Connect a P-ch MOSFET:\n- ANODE to Source\n- CATHODE to Drain\n- GATE to Gate"
+		(exclude_from_sim no)
+		(at 135.128 67.31 0)
+		(effects
+			(font
+				(size 1.27 1.27)
+			)
+			(justify left)
+		)
+	)
 	(junction
 		(at 142.24 100.33)
@@
 			(width 0)
 			(type default)
-		)
-	)
-	(text "Ideal diode controller\n\nUse a P-channel MOSFET as an ideal diode\nwith a very low voltage drop while maintaining\nreverse voltage protection and reverse current\nblocking."
-		(exclude_from_sim no)
-		(at 64.516 100.838 0)
-		(effects
-			(font
-				(size 1.27 1.27)
-			)
-			(justify left)
-		)
-	)
-	(text "Connect a P-ch MOSFET:\n- ANODE to Source\n- CATHODE to Drain\n- GATE to Gate"
-		(exclude_from_sim no)
-		(at 135.128 67.31 0)
-		(effects
-			(font
-				(size 1.27 1.27)
-			)
-			(justify left)
 		)
 	)
@@
 			)
 		)
+		(property "Characteristics" ""
+			(at 154.94 109.22 0)
+			(effects
+				(font
+					(size 1.27 1.27)
+				)
+				(hide yes)
+			)
+		)
+		(property "Sim.Enable" ""
+			(at 154.94 109.22 0)
+			(effects
+				(font
+					(size 1.27 1.27)
+				)
+			)
+		)
 		(pin "2"
 		)
@@
 			)
 		)
+		(property "Characteristics" ""
+			(at 134.62 109.22 0)
+			(effects
+				(font
+					(size 1.27 1.27)
+				)
+				(hide yes)
+			)
+		)
+		(property "Sim.Enable" ""
+			(at 134.62 109.22 0)
+			(effects
+				(font
+					(size 1.27 1.27)
+				)
+			)
+		)
 		(pin "2"
 		)
@@
 			)
 		)
+		(property "Characteristics" ""
+			(at 152.4 92.71 0)
+			(effects
+				(font
+					(size 1.27 1.27)
+				)
+				(hide yes)
+			)
+		)
+		(property "LCSC" "C2919802"
+			(at 152.4 92.71 0)
+			(effects
+				(font
+					(size 1.27 1.27)
+				)
+			)
+		)
+		(property "Sim.Enable" ""
+			(at 152.4 92.71 0)
+			(effects
+				(font
+					(size 1.27 1.27)
+				)
+			)
+		)
 		(pin "6"
 		)
@@
 			)
 		)
+		(property "Characteristics" ""
+			(at 137.16 92.71 0)
+			(effects
+				(font
+					(size 1.27 1.27)
+				)
+				(hide yes)
+			)
+		)
+		(property "LCSC" "C2919802"
+			(at 137.16 92.71 0)
+			(effects
+				(font
+					(size 1.27 1.27)
+				)
+			)
+		)
+		(property "Sim.Enable" ""
+			(at 137.16 92.71 0)
+			(effects
+				(font
+					(size 1.27 1.27)
+				)
+			)
+		)
