File: usb3if.kicad_sch (KiCad schematic)
At the start: 13 parts, among them J401 USB3_A, U401 AP2552W6-7, U402 RCLAMP0524P, U403 RCLAMP0524P

Commit message: Fix schematic ERC errors
Parts:
- U402, U403: footprint Package_SON:USON-10_2.5x1.0mm_P0.5mm -> Package_DFN_QFN:Diodes_UDFN-10_1.0x2.5mm_P0.5mm; symbol Yellow:TPD4EUSB30 -> Hatlabs:RCLAMP0524P
Connections:
- net SSTX+: no longer U402.7 (D2+)
- net SSTX-: no longer U402.6 (D2-)
- net USB3.D+: no longer U403.9 (D1-)
- net USB3.D-: no longer U403.10 (D1+)
- net USB3.RX+: no longer U403.7 (D2+)
- net USB3.RX-: no longer U403.6 (D2-)
- net VBUS_: no longer U402.9 (D1-)
- net at U402.1: no longer U402.10 (D1+)
Changed lines of the file:
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@@
-			)
-		)
-		(property "Sim.Enable" ""
-			(at 107.95 85.09 0)
-			(effects
-				(font
-					(size 1.27 1.27)
-				)
 			)
 		)
@@
 			)
 		)
-		(property "Sim.Enable" ""
-			(at 128.27 87.63 0)
-			(effects
-				(font
-					(size 1.27 1.27)
-				)
-			)
-		)
 		(pin "1"
 		)
@@
 			)
 		)
-		(property "Sim.Enable" ""
-			(at 78.74 139.7 0)
-			(effects
-				(font
-					(size 1.27 1.27)
-				)
-			)
-		)
 		(pin "1"
 		)
@@
 	)
 	(symbol
-		(lib_name "Power_Protection:TPD4EUSB30_1")
-		(lib_id "Yellow:TPD4EUSB30")
+		(lib_id "Hatlabs:RCLAMP0524P")
 		(at 218.44 130.81 0)
 		(unit 1)
@@
 			)
 		)
-		(property "Footprint" "Package_SON:USON-10_2.5x1.0mm_P0.5mm"
+		(property "Footprint" "Package_DFN_QFN:Diodes_UDFN-10_1.0x2.5mm_P0.5mm"
 			(at 194.31 140.97 0)
 			(effects
@@
 			)
 		)
-		(property "Description" ""
+		(property "Description" "4-Channel Low Capacitance TVS Diode Array, DFN-10"
 			(at 218.44 130.81 0)
 			(effects
@@
 					(size 1.27 1.27)
 				)
-			)
-		)
-		(property "Sim.Enable" ""
-			(at 218.44 130.81 0)
-			(effects
-				(font
-					(size 1.27 1.27)
-				)
+				(hide yes)
 			)
 		)
@@
 			)
 		)
-		(property "Sim.Enable" ""
-			(at 92.71 97.79 0)
-			(effects
-				(font
-					(size 1.27 1.27)
-				)
-			)
-		)
 		(pin "1"
 		)
@@
 			)
 		)
-		(property "Sim.Enable" ""
-			(at 193.04 76.2 0)
-			(effects
-				(font
-					(size 1.27 1.27)
-				)
-			)
-		)
 		(pin "1"
 		)
@@
 				)
 				(hide yes)
-			)
-		)
-		(property "Sim.Enable" ""
-			(at 200.66 96.52 0)
-			(effects
-				(font
-					(size 1.27 1.27)
-				)
 			)
 		)
@@
 			)
 		)
-		(property "Sim.Enable" ""
-			(at 220.98 86.36 0)
-			(effects
-				(font
-					(size 1.27 1.27)
-				)
-			)
-		)
 		(pin "10"
 		)
@@
 			)
 		)
-		(property "Sim.Enable" ""
-			(at 200.66 100.33 0)
-			(effects
-				(font
-					(size 1.27 1.27)
-				)
-			)
-		)
 		(pin "2"
 		)
@@
 	)
 	(symbol
-		(lib_name "Power_Protection:TPD4EUSB30_1")
-		(lib_id "Yellow:TPD4EUSB30")
+		(lib_id "Hatlabs:RCLAMP0524P")
 		(at 172.72 130.81 0)
 		(unit 1)
@@
 			)
 		)
-		(property "Footprint" "Package_SON:USON-10_2.5x1.0mm_P0.5mm"
+		(property "Footprint" "Package_DFN_QFN:Diodes_UDFN-10_1.0x2.5mm_P0.5mm"
 			(at 148.59 140.97 0)
 			(effects
@@
 			)
 		)
-		(property "Description" ""
+		(property "Description" "4-Channel Low Capacitance TVS Diode Array, DFN-10"
 			(at 172.72 130.81 0)
 			(effects
@@
 					(size 1.27 1.27)
 				)
-			)
-		)
-		(property "Sim.Enable" ""
-			(at 172.72 130.81 0)
-			(effects
-				(font
-					(size 1.27 1.27)
-				)
+				(hide yes)
 			)
 		)
@@
 				)
 				(hide yes)
-			)
-		)
-		(property "Sim.Enable" ""
-			(at 72.39 86.36 0)
-			(effects
-				(font
-					(size 1.27 1.27)
-				)
 			)
 		)
@@
 			)
 		)
-		(property "Sim.Enable" ""
-			(at 90.17 140.97 0)
-			(effects
-				(font
-					(size 1.27 1.27)
-				)
-			)
-		)
 		(pin "2"
 		)
@@
 			)
 		)
-		(property "Sim.Enable" ""
-			(at 78.74 132.08 0)
-			(effects
-				(font
-					(size 1.27 1.27)
-				)
-			)
-		)

Commit message: Renumber all sheets
Parts:
- renumbered C401 to C2501, C402 to C2502, C403 to C2503, C404 to C2504, D501 to D2401, D2402 to D2405, FB401 to FB2501, J401 to J2501, R502 to R2403, R401 to R2501, U401 to U2501, U402 to U2502, U403 to U2503
Changed lines of the file:
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@@
 		(on_board yes)
 		(dnp no)
-		(property "Reference" "#PWR0402"
+		(property "Reference" "#PWR02502"
 			(at 72.39 96.52 0)
 			(effects
@@
 		(dnp no)
 		(fields_autoplaced yes)
-		(property "Reference" "U401"
+		(property "Reference" "U2501"
 			(at 107.95 73.66 0)
 			(effects
@@
 		(dnp no)
 		(fields_autoplaced yes)
-		(property "Reference" "C402"
+		(property "Reference" "C2502"
 			(at 132.08 85.4709 0)
 			(effects
@@
 		(on_board yes)
 		(dnp no)
-		(property "Reference" "#PWR0403"
+		(property "Reference" "#PWR02503"
 			(at 128.27 97.79 0)
 			(effects
@@
 		(dnp no)
 		(fields_autoplaced yes)
-		(property "Reference" "#PWR0406"
+		(property "Reference" "#PWR02506"
 			(at 223.52 113.03 0)
 			(effects
@@
 		(on_board yes)
 		(dnp no)
-		(property "Reference" "#PWR02509"
+		(property "Reference" "#PWR02512"
 			(at 90.17 151.13 0)
 			(effects
@@
 		(on_board yes)
 		(dnp no)
-		(property "Reference" "D2402"
+		(property "Reference" "D2405"
 			(at 78.994 146.05 0)
 			(effects
@@
 		(dnp no)
 		(fields_autoplaced yes)
-		(property "Reference" "#PWR0407"
+		(property "Reference" "#PWR02507"
 			(at 172.72 149.86 0)
 			(effects
@@
 		(dnp no)
 		(fields_autoplaced yes)
-		(property "Reference" "#PWR0401"
+		(property "Reference" "#PWR02501"
 			(at 67.31 85.09 0)
 			(effects
@@
 		(on_board yes)
 		(dnp no)
-		(property "Reference" "U403"
+		(property "Reference" "U2503"
 			(at 218.44 118.11 0)
 			(effects
@@
 		(dnp no)
 		(fields_autoplaced yes)
-		(property "Reference" "#FLG0401"
+		(property "Reference" "#FLG02501"
 			(at 205.74 74.295 0)
 			(effects
@@
 		(dnp no)
 		(fields_autoplaced yes)
-		(property "Reference" "R401"
+		(property "Reference" "R2501"
 			(at 95.25 96.5199 0)
 			(effects
@@
 		(dnp no)
 		(fields_autoplaced yes)
-		(property "Reference" "FB401"
+		(property "Reference" "FB2501"
 			(at 193.0019 69.85 90)
 			(effects
@@
 		(on_board yes)
 		(dnp no)
-		(property "Reference" "C403"
+		(property "Reference" "C2503"
 			(at 200.6663 90.17 90)
 			(effects
@@
 		(dnp no)
 		(fields_autoplaced yes)
-		(property "Reference" "#PWR0408"
+		(property "Reference" "#PWR02508"
 			(at 218.44 149.86 0)
 			(effects
@@
 		(on_board yes)
 		(dnp no)
-		(property "Reference" "J401"
+		(property "Reference" "J2501"
 			(at 232.41 85.7249 0)
 			(effects
@@
 		(on_board yes)
 		(dnp no)
-		(property "Reference" "C404"
+		(property "Reference" "C2504"
 			(at 200.6663 106.68 90)
 			(effects
@@
 		(on_board yes)
 		(dnp no)
-		(property "Reference" "U402"
+		(property "Reference" "U2502"
 			(at 172.72 118.11 0)
 			(effects
@@
 		(on_board yes)
 		(dnp no)
-		(property "Reference" "C401"
+		(property "Reference" "C2501"
 			(at 75.311 85.1916 0)
 			(effects
@@
 		(on_board yes)
 		(dnp no)
-		(property "Reference" "#PWR0404"
+		(property "Reference" "#PWR02504"
 			(at 107.95 101.6 0)
 			(effects
@@
 		(dnp no)
 		(fields_autoplaced yes)
-		(property "Reference" "R502"
+		(property "Reference" "R2403"
 			(at 92.71 139.6999 0)
 			(effects
@@
 		(on_board yes)
 		(dnp no)
-		(property "Reference" "D501"
+		(property "Reference" "D2401"
 			(at 78.994 125.73 0)
 			(effects
@@
 		(on_board yes)
 		(dnp no)
-		(property "Reference" "#PWR0405"
+		(property "Reference" "#PWR02505"
 			(at 92.71 110.49 0)
 			(effects

Commit message: Reannotate components
Parts:
- renumbered D2401 to D2501, D2405 to D2502, R2403 to R2501, R2501 to R2502

Commit message: Most DRC errors fixed
Connections:
- net SSTX+: now also U2502.7 (NC)
- net SSTX-: now also U2502.6 (NC)
- net USB3.D+: now also U2503.9 (NC)
- net USB3.D-: now also U2503.10 (NC)
- net USB3.RX+: now also U2503.7 (NC)
- net USB3.RX-: now also U2503.6 (NC)
- net VBUS_: now also U2502.9 (NC)
- net at U2502.1: now also U2502.10 (NC)

Commit message: Fix most DRC errors, partial silk screen
Changed lines of the file:
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@@
 					(size 1.27 1.27)
 				)
+				(hide yes)
 			)
 		)

Commit message: Further refinements
Parts:
- removed D2501, D2502: RB521S-30, Diode_SMD:D_SOD-523, symbol Device:D_Schottky_Small
- added D2503: BAT54C,215, Package_TO_SOT_SMD:SOT-23, symbol Diode:BAT54C
Connections:
- net DIS: now also D2503.2
- net ~{ENAND}: now also D2503.3
- net ~{EN}: now also D2503.1
