File: usb3if.kicad_sch (KiCad schematic)
At the start: 12 parts, among them J2501 USB3_A, U2501 AP22652W6-7, U2502 RCLAMP0524P, U2503 RCLAMP0524P

Commit message: Reannotate the board
Parts:
- renumbered C2501 to C80, C2502 to C81, C2503 to C82, C2504 to C83, D2501 to D22, FB2501 to FB1, J2501 to J21, R2501 to R66, R2502 to R67, U2501 to U30, U2502 to U31, U2503 to U32

Commit message: Add GND/3.3V/5V headers, add missing JLC part numbers
Parts:
- added TP48, TP52, TP56, TP60: TestPoint, TestPoint:TestPoint_Pad_D1.0mm, symbol Connector:TestPoint
Connections:
- net DIS: now also TP52.1
- net VBUS_: now also TP60.1
- net ~{ENAND}: now also TP56.1
- net ~{EN}: now also TP48.1

Commit message: FInal v0.2.0 proto changes
Parts:
- renumbered C80 to C82, C81 to C83, C82 to C84, C83 to C85, FB1 to FB3, TP52 to TP38, TP48 to TP39, TP56 to TP40, TP60 to TP41

Commit message: Nailed the current limiter design
Also added more GND test pads
Also fixed the MCU I2C pinout
Parts:
- renumbered D22 to D23
