File: buck_3.3V.kicad_sch (KiCad schematic)
At the start: 16 parts, among them J4 3.3V Header, Q6 ASDM20N12ZB, U7 TPS566238PRQFR

Commit message: Remove unnecessary pullup
Parts:
- removed R30: 100k, Resistor_SMD:R_0402_1005Metric, symbol Device:R_Small
Connections:
- no-connect marks 1 -> 2
Changed lines of the file:
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@@
-	)
-	(junction
-		(at 74.93 74.93)
-		(diameter 0)
-		(color 0 0 0 0)
 	)
 	(junction
@@
 		(at 86.36 80.01)
 	)
+	(no_connect
+		(at 86.36 85.09)
+	)
 	(wire
 		(pts
@@
 	(wire
 		(pts
-			(xy 74.93 74.93) (xy 74.93 85.09)
-		)
-		(stroke
-			(width 0)
-			(type default)
-		)
-	)
-	(wire
-		(pts
 			(xy 82.55 64.77) (xy 86.36 64.77)
 		)
@@
 	(wire
 		(pts
-			(xy 82.55 85.09) (xy 86.36 85.09)
-		)
-		(stroke
-			(width 0)
-			(type default)
-		)
-	)
-	(wire
-		(pts
 			(xy 256.54 69.85) (xy 274.32 69.85)
 		)
@@
 	(wire
 		(pts
-			(xy 59.69 74.93) (xy 74.93 74.93)
-		)
-		(stroke
-			(width 0)
-			(type default)
-		)
-	)
-	(wire
-		(pts
 			(xy 256.54 44.45) (xy 256.54 69.85)
 		)
@@
 	(wire
 		(pts
-			(xy 74.93 74.93) (xy 86.36 74.93)
+			(xy 59.69 74.93) (xy 86.36 74.93)
 		)
 		(stroke
@@
 		(pts
 			(xy 59.69 74.93) (xy 59.69 83.82)
-		)
-		(stroke
-			(width 0)
-			(type default)
-		)
-	)
-	(wire
-		(pts
-			(xy 74.93 85.09) (xy 77.47 85.09)
 		)
 		(stroke
@@
 		(property "Netclass" "Analog"
 			(at 78.359 72.39 0)
-			(effects
-				(font
-					(size 1.27 1.27)
-					(italic yes)
-				)
-				(justify left)
-				(hide yes)
-			)
-		)
-	)
-	(netclass_flag ""
-		(length 2.54)
-		(shape round)
-		(at 85.09 85.09 0)
-		(fields_autoplaced yes)
-		(effects
-			(font
-				(size 1.27 1.27)
-			)
-			(justify left bottom)
-		)
-		(property "Netclass" "Digital"
-			(at 85.979 82.55 0)
 			(effects
 				(font
@@
 					(unit 1)
 				)
-			)
-		)
-	)
-	(symbol
-		(lib_id "Device:R_Small")
-		(at 80.01 85.09 270)
-		(unit 1)
-		(exclude_from_sim no)
-		(in_bom yes)
-		(on_board yes)
-		(dnp no)
-		(property "Reference" "R30"
-			(at 81.026 87.376 90)
-			(effects
-				(font
-					(size 1.27 1.27)
-				)
-			)
-		)
-		(property "Value" "100k"
-			(at 81.026 89.916 90)
-			(effects
-				(font
-					(size 1.27 1.27)
-				)
-			)
-		)
-		(property "Footprint" "Resistor_SMD:R_0402_1005Metric"
-			(at 80.01 85.09 0)
-			(effects
-				(font
-					(size 1.27 1.27)
-				)
-				(hide yes)
-			)
-		)
-		(property "Datasheet" "~"
-			(at 80.01 85.09 0)
-			(effects
-				(font
-					(size 1.27 1.27)
-				)
-				(hide yes)
-			)
-		)
-		(property "Description" "Resistor, small symbol"
-			(at 80.01 85.09 0)
-			(effects
-				(font
-					(size 1.27 1.27)
-				)
-				(hide yes)
-			)
-		)
-		(property "LCSC" "C25741"
-			(at 80.01 85.09 0)
-			(effects
-				(font
-					(size 1.27 1.27)
-				)
-				(hide yes)
-			)
-		)
-		(pin "1"
-		)
-		(pin "2"
-		)
-		(instances
-			(project "HALPI2"
-				(path "/abc482bd-3f17-4d35-80db-1da3dcdb5c27/c7bf4e1f-6bd1-4be7-9e56-1bd438bf5d42/e9d5ec1c-aaca-4440-9248-34d6a57da48f"
-					(reference "R30")
-					(unit 1)
-				)
