File: USB2.kicad_sch (KiCad schematic)
At the start: 5 parts, among them J3201 USB_C_Receptacle_USB2.0, U3201 RCLAMP0524P

Commit message: Reannotate the board
Parts:
- renumbered J3201 to J27, R3201 to R97, R3202 to R98, R3203 to R99, U3201 to U44
Changed lines of the file:
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@@
 		(on_board yes)
 		(dnp no)
-		(property "Reference" "#PWR03202"
+		(property "Reference" "#PWR0257"
 			(at 130.81 73.66 0)
 			(effects
@@
 			(project "HALPI2"
 				(path "/abc482bd-3f17-4d35-80db-1da3dcdb5c27/aa1d8d83-5167-420c-9ee7-3e4dcc942bfc"
-					(reference "#PWR03202")
+					(reference "#PWR0257")
 					(unit 1)
 				)
@@
 		(on_board yes)
 		(dnp no)
-		(property "Reference" "R3203"
+		(property "Reference" "R99"
 			(at 138.43 70.9868 90)
 			(effects
@@
 			(project "HALPI2"
 				(path "/abc482bd-3f17-4d35-80db-1da3dcdb5c27/aa1d8d83-5167-420c-9ee7-3e4dcc942bfc"
-					(reference "R3203")
+					(reference "R99")
 					(unit 1)
 				)
@@
 		(dnp no)
 		(fields_autoplaced yes)
-		(property "Reference" "#PWR03204"
+		(property "Reference" "#PWR0259"
 			(at 165.1 106.68 0)
 			(effects
@@
 			(project "HALPI2"
 				(path "/abc482bd-3f17-4d35-80db-1da3dcdb5c27/aa1d8d83-5167-420c-9ee7-3e4dcc942bfc"
-					(reference "#PWR03204")
+					(reference "#PWR0259")
 					(unit 1)
 				)
@@
 		(on_board yes)
 		(dnp no)
-		(property "Reference" "#PWR03205"
+		(property "Reference" "#PWR0260"
 			(at 172.72 106.68 0)
 			(effects
@@
 			(project "HALPI2"
 				(path "/abc482bd-3f17-4d35-80db-1da3dcdb5c27/aa1d8d83-5167-420c-9ee7-3e4dcc942bfc"
-					(reference "#PWR03205")
+					(reference "#PWR0260")
 					(unit 1)
 				)
@@
 		(on_board yes)
 		(dnp no)
-		(property "Reference" "U3201"
+		(property "Reference" "U44"
 			(at 163.83 109.22 0)
 			(effects
@@
 			(project "HALPI2"
 				(path "/abc482bd-3f17-4d35-80db-1da3dcdb5c27/aa1d8d83-5167-420c-9ee7-3e4dcc942bfc"
-					(reference "U3201")
+					(reference "U44")
 					(unit 1)
 				)
@@
 		(dnp no)
 		(fields_autoplaced yes)
-		(property "Reference" "R3201"
+		(property "Reference" "R97"
 			(at 121.92 64.7699 0)
 			(effects
@@
 			(project "HALPI2"
 				(path "/abc482bd-3f17-4d35-80db-1da3dcdb5c27/aa1d8d83-5167-420c-9ee7-3e4dcc942bfc"
-					(reference "R3201")
+					(reference "R97")
 					(unit 1)
 				)
@@
 		(on_board yes)
 		(dnp no)
-		(property "Reference" "#PWR03201"
+		(property "Reference" "#PWR0256"
 			(at 119.38 77.47 0)
 			(effects
@@
 			(project "HALPI2"
 				(path "/abc482bd-3f17-4d35-80db-1da3dcdb5c27/aa1d8d83-5167-420c-9ee7-3e4dcc942bfc"
-					(reference "#PWR03201")
+					(reference "#PWR0256")
 					(unit 1)
 				)
@@
 		(on_board yes)
 		(dnp no)
-		(property "Reference" "R3202"
+		(property "Reference" "R98"
 			(at 138.43 63.3668 90)
 			(effects
@@
 			(project "HALPI2"
 				(path "/abc482bd-3f17-4d35-80db-1da3dcdb5c27/aa1d8d83-5167-420c-9ee7-3e4dcc942bfc"
-					(reference "R3202")
+					(reference "R98")
 					(unit 1)
 				)
@@
 		(on_board yes)
 		(dnp no)
-		(property "Reference" "J3201"
+		(property "Reference" "J27"
 			(at 161.29 53.34 0)
 			(effects
@@
 			(project "HALPI2"
 				(path "/abc482bd-3f17-4d35-80db-1da3dcdb5c27/aa1d8d83-5167-420c-9ee7-3e4dcc942bfc"
-					(reference "J3201")
+					(reference "J27")
 					(unit 1)
 				)
@@
 		(on_board yes)
 		(dnp no)
-		(property "Reference" "#PWR03203"
+		(property "Reference" "#PWR0258"
 			(at 163.83 140.97 0)
 			(effects
@@
 			(project "HALPI2"
 				(path "/abc482bd-3f17-4d35-80db-1da3dcdb5c27/aa1d8d83-5167-420c-9ee7-3e4dcc942bfc"
-					(reference "#PWR03203")
-					(unit 1)
-				)
+					(reference "#PWR0258")
+					(unit 1)
+				)
