File: temp_sensor.kicad_sch (KiCad schematic)
At the start: 2 parts, among them U3801 TMP112xxDRL

Commit message: Reannotate the board
Parts:
- renumbered C3801 to C183, U3801 to U54
Changed lines of the file:
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@@
 		(dnp no)
 		(fields_autoplaced yes)
-		(property "Reference" "#PWR03802"
+		(property "Reference" "#PWR0343"
 			(at 140.97 69.85 0)
 			(effects
@@
 			(project ""
 				(path "/abc482bd-3f17-4d35-80db-1da3dcdb5c27/850df4bf-e40a-4082-adc2-76804638b949/9861be37-489a-48fe-bd2d-f1fa1d01f4aa"
-					(reference "#PWR03802")
+					(reference "#PWR0343")
 					(unit 1)
 				)
@@
 		(on_board yes)
 		(dnp no)
-		(property "Reference" "#PWR03801"
+		(property "Reference" "#PWR0342"
 			(at 129.54 74.93 0)
 			(effects
@@
 			(project "HALPI2"
 				(path "/abc482bd-3f17-4d35-80db-1da3dcdb5c27/850df4bf-e40a-4082-adc2-76804638b949/9861be37-489a-48fe-bd2d-f1fa1d01f4aa"
-					(reference "#PWR03801")
+					(reference "#PWR0342")
 					(unit 1)
 				)
@@
 		(dnp no)
 		(fields_autoplaced yes)
-		(property "Reference" "#PWR03803"
+		(property "Reference" "#PWR0344"
 			(at 140.97 102.87 0)
 			(effects
@@
 			(project ""
 				(path "/abc482bd-3f17-4d35-80db-1da3dcdb5c27/850df4bf-e40a-4082-adc2-76804638b949/9861be37-489a-48fe-bd2d-f1fa1d01f4aa"
-					(reference "#PWR03803")
+					(reference "#PWR0344")
 					(unit 1)
 				)
@@
 		(dnp no)
 		(fields_autoplaced yes)
-		(property "Reference" "C3801"
+		(property "Reference" "C183"
 			(at 133.35 60.96 90)
 			(effects
@@
 			(project "HALPI2"
 				(path "/abc482bd-3f17-4d35-80db-1da3dcdb5c27/850df4bf-e40a-4082-adc2-76804638b949/9861be37-489a-48fe-bd2d-f1fa1d01f4aa"
-					(reference "C3801")
+					(reference "C183")
 					(unit 1)
 				)
@@
 		(dnp no)
 		(fields_autoplaced yes)
-		(property "Reference" "U3801"
+		(property "Reference" "U54"
 			(at 156.21 74.8598 0)
 			(effects
@@
 			(project ""
 				(path "/abc482bd-3f17-4d35-80db-1da3dcdb5c27/850df4bf-e40a-4082-adc2-76804638b949/9861be37-489a-48fe-bd2d-f1fa1d01f4aa"
-					(reference "U3801")
-					(unit 1)
-				)
+					(reference "U54")
+					(unit 1)
+				)

Commit message: Fix DRC issues
Parts:
- U54: Component Class (none) -> fine_pitch
Changed lines of the file:
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@@
+			)
+		)
+		(property "Field8" ""
+			(at 133.35 68.58 0)
+			(effects
+				(font
+					(size 1.27 1.27)
+				)
+			)
+		)
+		(property "PartNumber" ""
+			(at 133.35 68.58 0)
+			(effects
+				(font
+					(size 1.27 1.27)
+				)
+			)
+		)
+		(property "Sim.Enable" ""
+			(at 133.35 68.58 0)
+			(effects
+				(font
+					(size 1.27 1.27)
+				)
 			)
 		)
@@
 			)
 		)
-		(property "LCSC Part" ""
+		(property "JLCPCB_CORRECTION" "0;0;180"
+			(at 140.97 86.36 0)
+			(effects
+				(font
+					(size 1.27 1.27)
+				)
+				(hide yes)
+			)
+		)
+		(property "PartNumber" ""
 			(at 140.97 86.36 0)
 			(effects
@@
 			)
 		)
-		(property "JLCPCB_CORRECTION" "0;0;180"
+		(property "Sim.Enable" ""
 			(at 140.97 86.36 0)
 			(effects
+				(font
+					(size 1.27 1.27)
+				)
+			)
+		)
+		(property "Component Class" "fine_pitch"
+			(at 140.97 86.36 0)
+			(effects

Commit message: FInal v0.2.0 proto changes
Parts:
- renumbered C183 to C186
Changed lines of the file:
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@@
 		(dnp no)
 		(fields_autoplaced yes)
-		(property "Reference" "#PWR0343"
+		(property "Reference" "#PWR0363"
 			(at 140.97 69.85 0)
 			(effects
@@
 			(project ""
 				(path "/abc482bd-3f17-4d35-80db-1da3dcdb5c27/850df4bf-e40a-4082-adc2-76804638b949/9861be37-489a-48fe-bd2d-f1fa1d01f4aa"
-					(reference "#PWR0343")
+					(reference "#PWR0363")
 					(unit 1)
 				)
@@
 		(on_board yes)
 		(dnp no)
-		(property "Reference" "#PWR0342"
+		(property "Reference" "#PWR0362"
 			(at 129.54 74.93 0)
 			(effects
@@
 			(project "HALPI2"
 				(path "/abc482bd-3f17-4d35-80db-1da3dcdb5c27/850df4bf-e40a-4082-adc2-76804638b949/9861be37-489a-48fe-bd2d-f1fa1d01f4aa"
-					(reference "#PWR0342")
+					(reference "#PWR0362")
 					(unit 1)
 				)
@@
 		(dnp no)
 		(fields_autoplaced yes)
-		(property "Reference" "#PWR0344"
+		(property "Reference" "#PWR0364"
 			(at 140.97 102.87 0)
 			(effects
@@
 			(project ""
 				(path "/abc482bd-3f17-4d35-80db-1da3dcdb5c27/850df4bf-e40a-4082-adc2-76804638b949/9861be37-489a-48fe-bd2d-f1fa1d01f4aa"
-					(reference "#PWR0344")
+					(reference "#PWR0364")
 					(unit 1)
 				)
@@
 		(dnp no)
 		(fields_autoplaced yes)
-		(property "Reference" "C183"
+		(property "Reference" "C186"
 			(at 133.35 60.96 90)
 			(effects
@@
 			(project "HALPI2"
 				(path "/abc482bd-3f17-4d35-80db-1da3dcdb5c27/850df4bf-e40a-4082-adc2-76804638b949/9861be37-489a-48fe-bd2d-f1fa1d01f4aa"
-					(reference "C183")
+					(reference "C186")
 					(unit 1)
 				)
@@
 			)
 		)
+		(property "Component Class" "fine_pitch"
+			(at 140.97 86.36 0)
+			(effects
+				(font
+					(size 1.27 1.27)
+				)
+				(hide yes)
+			)
+		)
 		(property "Sim.Enable" ""
 			(at 140.97 86.36 0)
@@
 			)
 		)
-		(property "Component Class" "fine_pitch"
-			(at 140.97 86.36 0)
-			(effects
-				(font
-					(size 1.27 1.27)
-				)
-				(hide yes)
-			)
-		)

Commit message: Nailed the current limiter design
Also added more GND test pads
Also fixed the MCU I2C pinout
Parts:
- U54: value TMP112xxDRL -> TMP112AIDRL
Changed lines of the file:
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@@
 		(dnp no)
 		(fields_autoplaced yes)
-		(property "Reference" "#PWR0363"
+		(property "Reference" "#PWR0362"
 			(at 140.97 69.85 0)
 			(effects
@@
 			(project ""
 				(path "/abc482bd-3f17-4d35-80db-1da3dcdb5c27/850df4bf-e40a-4082-adc2-76804638b949/9861be37-489a-48fe-bd2d-f1fa1d01f4aa"
-					(reference "#PWR0363")
+					(reference "#PWR0362")
 					(unit 1)
 				)
@@
 		(on_board yes)
 		(dnp no)
-		(property "Reference" "#PWR0362"
+		(property "Reference" "#PWR0361"
 			(at 129.54 74.93 0)
 			(effects
@@
 			(project "HALPI2"
 				(path "/abc482bd-3f17-4d35-80db-1da3dcdb5c27/850df4bf-e40a-4082-adc2-76804638b949/9861be37-489a-48fe-bd2d-f1fa1d01f4aa"
-					(reference "#PWR0362")
+					(reference "#PWR0361")
 					(unit 1)
 				)
@@
 		(dnp no)
 		(fields_autoplaced yes)
-		(property "Reference" "#PWR0364"
+		(property "Reference" "#PWR0363"
 			(at 140.97 102.87 0)
 			(effects
@@
 			(project ""
 				(path "/abc482bd-3f17-4d35-80db-1da3dcdb5c27/850df4bf-e40a-4082-adc2-76804638b949/9861be37-489a-48fe-bd2d-f1fa1d01f4aa"
-					(reference "#PWR0364")
+					(reference "#PWR0363")
 					(unit 1)
 				)
@@
 			)
 		)
-		(property "LCSC Part" ""
-			(at 133.35 68.58 0)
-			(effects
-				(font
-					(size 1.27 1.27)
-				)
-			)
-		)
-		(property "Field8" ""
-			(at 133.35 68.58 0)
-			(effects
-				(font
-					(size 1.27 1.27)
-				)
-			)
-		)
-		(property "PartNumber" ""
-			(at 133.35 68.58 0)
-			(effects
-				(font
-					(size 1.27 1.27)
-				)
-			)
-		)
 		(pin "1"
 		)
@@
 			)
 		)
-		(property "Value" "TMP112xxDRL"
+		(property "Value" "TMP112AIDRL"
 			(at 156.21 77.3998 0)
 			(effects
@@
 			)
 		)
-		(property "PartNumber" ""
-			(at 140.97 86.36 0)
-			(effects
-				(font
-					(size 1.27 1.27)
-				)
-			)
-		)

Commit message: Final chores
- Reannotate components
- Improve USB2 connector skew matching
- Update sheet blocks
- Fix some diff-pair double-inversions
Parts:
- renumbered C186 to C184, U54 to U53
Changed lines of the file:
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@@
 	(title_block
 		(title "HALPI2")
-		(date "2025-03-27")
-		(rev "v0.2.0")
+		(date "2025-05-08")
+		(rev "v0.3.0")
 		(company "Hat Labs Oy")
 		(comment 1 "https://ohwr.org/cern_ohl_s_v2.pdf")
@@
 		(dnp no)
 		(fields_autoplaced yes)
-		(property "Reference" "#PWR0362"
+		(property "Reference" "#PWR0356"
 			(at 140.97 69.85 0)
 			(effects
@@
 			(project ""
 				(path "/abc482bd-3f17-4d35-80db-1da3dcdb5c27/850df4bf-e40a-4082-adc2-76804638b949/9861be37-489a-48fe-bd2d-f1fa1d01f4aa"
-					(reference "#PWR0362")
+					(reference "#PWR0356")
 					(unit 1)
 				)
@@
 		(on_board yes)
 		(dnp no)
-		(property "Reference" "#PWR0361"
+		(property "Reference" "#PWR0355"
 			(at 129.54 74.93 0)
 			(effects
@@
 			(project "HALPI2"
 				(path "/abc482bd-3f17-4d35-80db-1da3dcdb5c27/850df4bf-e40a-4082-adc2-76804638b949/9861be37-489a-48fe-bd2d-f1fa1d01f4aa"
-					(reference "#PWR0361")
+					(reference "#PWR0355")
 					(unit 1)
 				)
@@
 		(dnp no)
 		(fields_autoplaced yes)
-		(property "Reference" "#PWR0363"
+		(property "Reference" "#PWR0357"
 			(at 140.97 102.87 0)
 			(effects
@@
 			(project ""
 				(path "/abc482bd-3f17-4d35-80db-1da3dcdb5c27/850df4bf-e40a-4082-adc2-76804638b949/9861be37-489a-48fe-bd2d-f1fa1d01f4aa"
-					(reference "#PWR0363")
+					(reference "#PWR0357")
 					(unit 1)
 				)
@@
 		(dnp no)
 		(fields_autoplaced yes)
-		(property "Reference" "C186"
+		(property "Reference" "C184"
 			(at 133.35 60.96 90)
 			(effects
@@
 			(project "HALPI2"
 				(path "/abc482bd-3f17-4d35-80db-1da3dcdb5c27/850df4bf-e40a-4082-adc2-76804638b949/9861be37-489a-48fe-bd2d-f1fa1d01f4aa"
-					(reference "C186")
+					(reference "C184")
 					(unit 1)
 				)
@@
 		(dnp no)
 		(fields_autoplaced yes)
-		(property "Reference" "U54"
+		(property "Reference" "U53"
 			(at 156.21 74.8598 0)
 			(effects
@@
 			(project ""
 				(path "/abc482bd-3f17-4d35-80db-1da3dcdb5c27/850df4bf-e40a-4082-adc2-76804638b949/9861be37-489a-48fe-bd2d-f1fa1d01f4aa"
-					(reference "U54")
+					(reference "U53")
 					(unit 1)
 				)
