File: PCIe.kicad_sch (KiCad schematic)
At the start: 12 parts, among them J25 Bus_M.2_Socket_M

Commit message: Re-route fast interfaces; split 3.3V to permanent and controller parts
Connections:
- net PCIe.CLK+: now also J25.55 (REFCLKp); no longer J25.53 (REFCLKn)
- net PCIe.CLK-: now also J25.53 (REFCLKn); no longer J25.55 (REFCLKp)
- net PCIe.TX+: now also J25.49 (PETp0/SATA-A+); no longer J25.47 (PETn0/SATA-A-)
- net PCIe.TX-: now also J25.47 (PETn0/SATA-A-); no longer J25.49 (PETp0/SATA-A+)
Changed lines of the file:
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@@
 	)
 	(label "PCIe.CLK-"
-		(at 76.2 127 0)
+		(at 76.2 129.54 0)
 		(effects
 			(font
@@
 	)
 	(label "PCIe.TX-"
-		(at 74.93 58.42 0)
+		(at 74.93 60.96 0)
 		(effects
 			(font
@@
 	)
 	(label "PCIe.TX+"
-		(at 74.93 60.96 0)
+		(at 74.93 58.42 0)
 		(effects
 			(font
@@
 	)
 	(label "PCIe.CLK+"
-		(at 76.2 129.54 0)
+		(at 76.2 127 0)
 		(effects
 			(font

Commit message: Add a clock oscillator for NVMe SUSCLK
Parts:
- added C16: 1uF, Capacitor_SMD:C_0402_1005Metric, symbol Device:C
- added C18, C802: 22pF C0G, Capacitor_SMD:C_0603_1608Metric, symbol Device:C_Small
- added R149: 1M, Resistor_SMD:R_0402_1005Metric, symbol Device:R
- added R150: 330k, Resistor_SMD:R_0603_1608Metric, symbol Device:R
- added TP94, TP95, TP96: TestPoint, TestPoint:TestPoint_Pad_D1.0mm, symbol Connector:TestPoint
- added U4: 74LVC1GU04, Package_TO_SOT_SMD:SOT-353_SC-70-5, symbol 74xGxx:74LVC1GU04
- added Y801: X1A000061000200, Crystal:Crystal_SMD_2012-2Pin_2.0x1.2mm, symbol Device:Crystal
Connections:
- net +3.3V: now also C16.1, U4.5 (VCC)
- net GND: now also C16.2, C18.1, C802.1, U4.3 (GND)
- net SUSCLK: now reaches J25.68 (SUSCLK)
- net SUSCLK: now also R150.2, TP94.1, U4.4
- new net OSCI: C802.2, R149.1, TP96.1, U4.2, Y801.2
- new net OSCO: C18.2, R149.2, R150.1, TP95.1, Y801.1
- no-connect marks 15 -> 14

Commit message: Bump board revision to 0.6.1.
Adjust M.2 connector SUSCLK direction.
Parts:
- J25: symbol Hatlabs:Bus_M.2_Socket_M -> HL_Connector:Bus_M.2_Socket_M
Changed lines of the file:
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@@
 	(title_block
 		(title "HALPI2")
-		(date "2025-10-07")
-		(rev "v0.6.0")
+		(date "2025-12-20")
+		(rev "v0.6.1")
 		(company "Hat Labs Oy")
 		(comment 1 "https://ohwr.org/cern_ohl_s_v2.pdf")
@@
 	)
 	(symbol
-		(lib_id "Hatlabs:Bus_M.2_Socket_M")
+		(lib_id "HL_Connector:Bus_M.2_Socket_M")
 		(at 114.3 91.44 0)
 		(unit 1)

Commit message: Update JLCPCB corrections
Parts:
- U4: JLCPCB_CORRECTION (none) -> 0;0;270
Changed lines of the file:
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@@
+			)
+		)
+		(property "JLCPCB_CORRECTION" "0;0;270"
+			(at 203.2 105.41 0)
+			(effects
+				(font
+					(size 1.27 1.27)
+				)
+				(hide yes)
 			)
 		)

Commit message: Increase the SUSCLK oscillator C1 cap value
Parts:
- C18: value 22pF C0G -> 100pF C0G; LCSC C1653 -> (none)
Other:
- note added: "Temporary fix: ensure the oscillator starts even with a fast 74LVC inverter."
Changed lines of the file:
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@@
+		)
+	)
+	(text "Temporary fix: ensure the oscillator starts\neven with a fast 74LVC inverter."
+		(exclude_from_sim no)
+		(at 220.98 146.05 0)
+		(effects
+			(font
+				(size 1.27 1.27)
+			)
+			(justify left)
 		)
 	)
@@
 			)
 		)
-		(property "Value" "22pF C0G"
+		(property "Value" "100pF C0G"
 			(at 212.09 146.0437 90)
 			(effects
@@
 			)
 		)
-		(property "LCSC" "C1653"
+		(property "LCSC" ""
 			(at 215.9 146.05 0)
 			(effects

Commit message: Fix v0.6.1 RS-485 issues
- Add a pulldown to ~{EN}
- Change ~{EN} to GPIO15
- Add pull-ups and pull-downs to TX pins
Parts:
- C18: LCSC (none) -> C14858
Changed lines of the file:
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@@
 			)
 		)
-		(property "LCSC" ""
+		(property "LCSC" "C14858"
 			(at 215.9 146.05 0)
 			(effects
